File: Hw/LoRA_USBStick.sch (KiCad schematic (older format))
At the start: 16 parts, among them J10 USB_B, J4 SWD, SW1 RST, U1 ATSAMD21E, U2 RFM95W-868S2, U3 AP2112K-3.3

Commit message: udpate version with u.fl connector
Parts:
- AE1: footprint agroin:SMA_EDGE -> Connectors:MOLEX_1661
Changed lines of the file:
@@
 F 0 "AE1" H 10780 1095 50  0000 R CNN
 F 1 "Antenna_Shield" H 11160 1170 50  0000 R CNN
-F 2 "agroin:SMA_EDGE" H 10855 1020 50  0001 C CNN
+F 2 "Connectors:MOLEX_1661" H 10855 1020 50  0001 C CNN
 F 3 "" H 10855 1020 50  0001 C CNN
 	1    10855 920
