File: Hw/LoRA_USBStick.sch (KiCad schematic (older format))
At the start: 16 parts, among them J10 USB_B, J4 SWD, SW1 RST, U1 ATSAMD21E, U2 RFM95W-868S2, U3 AP2112K-3.3

Commit message: fix part number micro
Parts:
- U1: manf# ATSAMD21E15B-AUT -> ATSAMD21E18A-U
Changed lines of the file:
@@
 F 2 "Housings_QFP:TQFP-32_7x7mm_Pitch0.8mm" H 5595 2615 20  0001 C CNN
 F 3 "" H 5565 2465 60  0001 C CNN
-F 4 "ATSAMD21E15B-AUT" H 5565 2465 60  0001 C CNN "manf#"
+F 4 "ATSAMD21E18A-U" H 5565 2465 60  0001 C CNN "manf#"
 	1    5565 2465
 	1    0    0    -1
