File: Hw/LoRA_USBStick.kicad_pcb (KiCad board)
At the start: 2 copper layers, 61.5 x 18.7 mm, 35 parts, among them J10 USB_B, SW3 RST, U1 RP2040, U2 RFM95W-868S2, U3 AP2112K-3.3, U4 W25Q16JV, Y1 12Mhz

Commit message: fix routing
Parts:
- moved C12 1.44 mm to (139.0, 106.5)
Routing:
- net +3V3: track 107.7 -> 130.5 mm
- net /DIO2: track 30.7 -> 33.6 mm
- net /RFM_RST: track 34.9 -> 36.3 mm
- net /DIO1: track 32.3 -> 33.5 mm
- net GND: track 24.5 -> 23.4 mm, vias 14 -> 13
- net /DIO0: track 36.2 -> 37.3 mm

Commit message: Add labels
Parts:
- added kibuzzard-62D459CC: G***, kibuzzard-62D459CC, B.Cu at (135.3, 116.7)
Other:
- board text removed: "3.3v"
- board text removed: "GND"
- board text removed: "SWCLK"
- board text removed: "SWDIO"

Commit message: update labels
Parts:
- moved G*** 2.60 mm to (162.3, 116.5)
Other:
- board text added: "USB-Stick V2.5 CatWAN RP2040"
- board text removed: "USB-Stick V2.4 CatWAN"
Changed lines of the file:
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@@
   )
   (footprint "Aesthetics:electronic_cats_logo_8x6" (layer "B.Cu")
-    (at 162.192 113.9224 180)
+    (at 162.27 116.52 180)
     (attr through_hole)
     (fp_text reference "G***" (at 0 0 180) (layer "B.SilkS") hide
@@
   (gr_line (start 178.2572 118.999) (end 176.53 118.999) (layer "Edge.Cuts") (width 0.2))
   (gr_line (start 178.2572 108.7628) (end 176.53 108.7628) (layer "Edge.Cuts") (width 0.2))
-  (gr_text "Compatible with \nLoRaWAN®" (at 162.192 120.6724) (layer "B.SilkS")
+  (gr_text "Compatible with \nLoRaWAN®" (at 162.19 121.73) (layer "B.SilkS")
+    (effects (font (size 1 1) (thickness 0.25)) (justify mirror))
+  )
+  (gr_text "USB-Stick V2.5\nCatWAN\nRP2040" (at 162.11 109.25) (layer "B.SilkS")
     (effects (font (size 1.5 1.5) (thickness 0.3)) (justify mirror))
   )
-  (gr_text "USB-Stick V2.4\nCatWAN" (at 162.142 107.5224) (layer "B.SilkS")
-    (effects (font (size 1.5 1.5) (thickness 0.3)) (justify mirror))
-  )

Commit message: update label v3.0
Other:
- board text added: "USB-Stick V3.0 CatWAN RP2040"
- board text removed: "USB-Stick V2.5 CatWAN RP2040"
Changed lines of the file:
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@@
     (effects (font (size 1 1) (thickness 0.25)) (justify mirror))
   )
-  (gr_text "USB-Stick V2.5\nCatWAN\nRP2040" (at 162.11 109.25) (layer "B.SilkS")
+  (gr_text "USB-Stick V3.0\nCatWAN\nRP2040" (at 162.11 109.25) (layer "B.SilkS")
     (effects (font (size 1.5 1.5) (thickness 0.3)) (justify mirror))
   )
