File: Hw/LoRA_USBStick.kicad_sch (KiCad schematic)
At the start: 35 parts

Commit message: PCB route
Parts:
- removed J4: (no value), symbol Connector:Conn_01x06_Female
- AE1: value (none) -> Antenna_Shield; footprint (none) -> agroin:SMA_EDGE
- C1, C3: value (none) -> 27pF; footprint (none) -> Capacitor_SMD:C_0603_1608Metric
- C10, C11, C12, C13, C14, C15, C16, C17, C4, C8: value (none) -> 0.1uF; footprint (none) -> Capacitor_SMD:C_0603_1608Metric
- C2, C9: value (none) -> 1uF; footprint (none) -> Capacitor_SMD:C_0603_1608Metric
- C5: value (none) -> 0.1uF; footprint (none) -> Capacitor_SMD:C_0805_2012Metric_Pad1.15x1.40mm_HandSolder
- C6, C7: value (none) -> 10uF; footprint (none) -> Capacitor_SMD:C_0805_2012Metric_Pad1.15x1.40mm_HandSolder
- D1: value (none) -> Rx; footprint (none) -> LED_SMD:LED_0805_2012Metric_Pad1.15x1.40mm_HandSolder
- D2: value (none) -> ON; footprint (none) -> LED_SMD:LED_0805_2012Metric_Pad1.15x1.40mm_HandSolder
- J10: value (none) -> USB_B; footprint (none) -> Connectors:C46394
- JP1: value (none) -> BOOT; footprint (none) -> Jumper:SolderJumper-2_P1.3mm_Open_Pad1.0x1.5mm
- R11, R9: value (none) -> 120R; footprint (none) -> Resistor_SMD:R_0805_2012Metric_Pad1.15x1.40mm_HandSolder
- R2: value (none) -> 1K; footprint (none) -> Resistor_SMD:R_0603_1608Metric
- R3, R4: value (none) -> 27; footprint (none) -> Resistor_SMD:R_0603_1608Metric
- R5: value (none) -> 10K; footprint (none) -> Resistor_SMD:R_0603_1608Metric
- SW3: value (none) -> RST; footprint (none) -> Button_Switch_SMD:SW_SPST_TL3342
- U1: value (none) -> RP2040; footprint (none) -> RP2040:RP2040-QFN-56
- U2: value (none) -> RFM95W-868S2; footprint (none) -> RF_Module:HOPERF_RFM9XW_SMD
- U3: value (none) -> AP2112K-3.3; footprint (none) -> Package_TO_SOT_SMD:SOT-23-5
- U4: value (none) -> W25Q16JV; footprint (none) -> RP2040:W25Q16JVUUIQ
- Y1: value (none) -> 12Mhz; footprint (none) -> Crystal:Crystal_SMD_5032-2Pin_5.0x3.2mm
Connections:
- net Rx_LED is gone; now on net RX_LED: R11.1
- net RX_LED: now also U1.37 (GPIO25); no longer U1.2 (GPIO0)
- net SWCLK: no longer names the net of U1.24 (SWCLK)
- net SWDIO: no longer names the net of U1.25 (SWD)
- no-connect marks 24 -> 23

Commit message: update floorplan and routing
Parts:
- R11, R9: footprint Resistor_SMD:R_0805_2012Metric_Pad1.15x1.40mm_HandSolder -> Resistor_SMD:R_0603_1608Metric
Changed lines of the file:
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@@
       (effects (font (size 1.27 1.27)) (justify left))
     )
-    (property "Footprint" "Resistor_SMD:R_0805_2012Metric_Pad1.15x1.40mm_HandSolder" (id 2) (at 80.01 77.851 0)
+    (property "Footprint" "Resistor_SMD:R_0603_1608Metric" (id 2) (at 80.01 77.851 0)
       (effects (font (size 1.27 1.27)) hide)
     )
@@
       (effects (font (size 1.27 1.27)) (justify left))
     )
-    (property "Footprint" "Resistor_SMD:R_0805_2012Metric_Pad1.15x1.40mm_HandSolder" (id 2) (at 62.103 78.486 0)
+    (property "Footprint" "Resistor_SMD:R_0603_1608Metric" (id 2) (at 62.103 78.486 0)
       (effects (font (size 1.27 1.27)) hide)
     )
@@
     )
     (path "/00000000-0000-0000-0000-00005b0d38e2"
-      (reference "R9") (unit 1) (value "120R") (footprint "Resistor_SMD:R_0805_2012Metric_Pad1.15x1.40mm_HandSolder")
+      (reference "R9") (unit 1) (value "120R") (footprint "Resistor_SMD:R_0603_1608Metric")
     )
     (path "/00000000-0000-0000-0000-00005b0d3e93"
-      (reference "R11") (unit 1) (value "120R") (footprint "Resistor_SMD:R_0805_2012Metric_Pad1.15x1.40mm_HandSolder")
+      (reference "R11") (unit 1) (value "120R") (footprint "Resistor_SMD:R_0603_1608Metric")
     )
     (path "/bd279f0b-459f-41ba-8171-ac9414a30ac1"

Commit message: Change a fototprint and routing
Parts:
- AE1: value Antenna_Shield -> (none); footprint agroin:SMA_EDGE -> (none)
- C1, C3: value 27pF -> (none); footprint Capacitor_SMD:C_0603_1608Metric -> (none)
- C10, C11, C12, C13, C14, C15, C16, C17, C4, C8: value 0.1uF -> (none); footprint Capacitor_SMD:C_0603_1608Metric -> (none)
- C2, C9: value 1uF -> (none); footprint Capacitor_SMD:C_0603_1608Metric -> (none)
- C5: value 0.1uF -> (none); footprint Capacitor_SMD:C_0805_2012Metric_Pad1.15x1.40mm_HandSolder -> (none)
- C6, C7: value 10uF -> (none); footprint Capacitor_SMD:C_0805_2012Metric_Pad1.15x1.40mm_HandSolder -> (none)
- D1: value Rx -> (none); footprint LED_SMD:LED_0805_2012Metric_Pad1.15x1.40mm_HandSolder -> (none)
- D2: value ON -> (none); footprint LED_SMD:LED_0805_2012Metric_Pad1.15x1.40mm_HandSolder -> (none)
- J10: value USB_B -> (none); footprint Connectors:C46394 -> (none)
- JP1: value BOOT -> (none); footprint Jumper:SolderJumper-2_P1.3mm_Open_Pad1.0x1.5mm -> (none)
- R11, R9: value 120R -> (none); footprint Resistor_SMD:R_0603_1608Metric -> (none)
- R2: value 1K -> (none); footprint Resistor_SMD:R_0603_1608Metric -> (none)
- R3, R4: value 27 -> (none); footprint Resistor_SMD:R_0603_1608Metric -> (none)
- R5: value 10K -> (none); footprint Resistor_SMD:R_0603_1608Metric -> (none)
- SW3: value RST -> (none); footprint Button_Switch_SMD:SW_SPST_TL3342 -> (none)
- U1: value RP2040 -> (none); footprint RP2040:RP2040-QFN-56 -> (none)
- U2: value RFM95W-868S2 -> (none); footprint RF_Module:HOPERF_RFM9XW_SMD -> (none)
- U3: value AP2112K-3.3 -> (none); footprint Package_TO_SOT_SMD:SOT-23-5 -> (none)
- U4: value W25Q16JV -> (none); footprint RP2040:W25Q16JVUUIQ -> (none)
- Y1: value 12Mhz -> (none); footprint Crystal:Crystal_SMD_5032-2Pin_5.0x3.2mm -> (none)

Commit message: BOM updated
Parts:
- AE1: value (none) -> Antenna_Shield; footprint (none) -> agroin:SMA_EDGE; LCSC# (none) -> C2913580
- C1, C3: value (none) -> 27pF; footprint (none) -> Capacitor_SMD:C_0603_1608Metric; manf# EC -> C0603C270J5GAC7411
- C10, C11, C12, C13, C14, C15, C16, C17, C4, C8: value (none) -> 0.1uF; footprint (none) -> Capacitor_SMD:C_0603_1608Metric; LCSC# (none) -> C282519; manf# EC -> (none)
- C2, C9: value (none) -> 1uF; footprint (none) -> Capacitor_SMD:C_0603_1608Metric; LCSC# (none) -> C711096; manf# EC -> (none)
- C5: value (none) -> 0.1uF; footprint (none) -> Capacitor_SMD:C_0805_2012Metric_Pad1.15x1.40mm_HandSolder
- C6, C7: value (none) -> 10uF; footprint (none) -> Capacitor_SMD:C_0805_2012Metric_Pad1.15x1.40mm_HandSolder; LCSC# (none) -> C1713; manf# GRM21BC80J106KE19L -> (none)
- D1: value (none) -> Rx; footprint (none) -> LED_SMD:LED_0805_2012Metric_Pad1.15x1.40mm_HandSolder
- D2: value (none) -> ON; footprint (none) -> LED_SMD:LED_0805_2012Metric_Pad1.15x1.40mm_HandSolder
- J10: value (none) -> USB_B; footprint (none) -> Connectors:C46394; LCSC# (none) -> C46394
- JP1: value (none) -> BOOT; footprint (none) -> Jumper:SolderJumper-2_P1.3mm_Open_Pad1.0x1.5mm; now not fitted
- R11, R9: value (none) -> 120R; footprint (none) -> Resistor_SMD:R_0603_1608Metric
- R2: value (none) -> 1K; footprint (none) -> Resistor_SMD:R_0603_1608Metric; LCSC# (none) -> C21190
- R3, R4: value (none) -> 27; footprint (none) -> Resistor_SMD:R_0603_1608Metric; LCSC# (none) -> C2907136
- R5: value (none) -> 10K; footprint (none) -> Resistor_SMD:R_0603_1608Metric; LCSC# (none) -> C2930027
- SW3: value (none) -> RST; footprint (none) -> Switches:C455281
- U1: value (none) -> RP2040; footprint (none) -> RP2040:RP2040-QFN-56; LCSC# (none) -> C2040
- U2: value (none) -> RFM95W-868S2; footprint (none) -> RF_Module:HOPERF_RFM9XW_SMD; manf# (none) -> 109990166
- U3: value (none) -> AP2112K-3.3; footprint (none) -> Package_TO_SOT_SMD:SOT-23-5; manf# (none) -> AP7365-33WG-7
- U4: value (none) -> W25Q16JV; footprint (none) -> RP2040:W25Q16JVUUIQ; manf# W25Q16JVUXIQ -> W25Q16JVUUIQTR
- Y1: value (none) -> 12Mhz; footprint (none) -> Crystal:Crystal_SMD_5032-2Pin_5.0x3.2mm
